File: JonoBro.kicad_pcb (KiCad board)
At the start: 2 copper layers, 44.7 x 56.5 mm, 37 parts, among them J1 Conn_01x02_Pin, J2 Conn_01x02_Pin, J3 Conn_01x02_Pin, J4 Conn_01x02_Pin, J5 Conn_01x06_Socket, Q1 CSD19537Q3, Q2 MMBT3904, Q3 CSD19537Q3, U1 AOZ1280CI, U2 ESP32-C3-MINI-1

Commit message: v0.1 submitted for PCBA
Parts:
- added FID1: Fiducial, Fiducial:Fiducial_0.5mm_Mask1.5mm, F.Cu at (121.5, 65.5)
- added FID2: Fiducial, Fiducial:Fiducial_0.5mm_Mask1.5mm, F.Cu at (160.0, 65.5)
- added FID3: Fiducial, Fiducial:Fiducial_0.5mm_Mask1.5mm, F.Cu at (160.5, 118.0)
- added FID4: Fiducial, Fiducial:Fiducial_0.5mm_Mask1.5mm, F.Cu at (122.5, 117.5)
- added G***: LOGO, Acea:ae_5mm, F.Cu at (138.0, 97.0)
- moved H1 1.18 mm to (144.0, 98.5)
Routing:
- net Net-(D4-A): vias 81 -> 79
- net +12V: vias 146 -> 141
Other:
- board text added: "JLCJLCJLCJLC"
