File: JonoBro.kicad_sch (KiCad schematic)
At the start: 9 parts, among them J1 Conn_01x02_Pin, J2 Conn_01x02_Pin, J3 Conn_01x02_Pin, J4 Conn_01x02_Pin, Q1 PSMN5R2-60YL, U1 ATtiny25V-10M, U2 HT75xx-1-SOT89

Commit message: seems good to me
Parts:
- removed C1, C2: 10uF, Capacitor_SMD:C_0603_1608Metric, symbol Device:C_Small
- removed Q1: PSMN5R2-60YL, Package_TO_SOT_SMD:LFPAK56, symbol Transistor_FET:PSMN5R2-60YL
- removed U1: ATtiny25V-10M, Package_DFN_QFN:QFN-20-1EP_4x4mm_P0.5mm_EP2.6x2.6mm, symbol MCU_Microchip_ATtiny:ATtiny25V-10M
- removed U2: HT75xx-1-SOT89, Package_TO_SOT_SMD:SOT-89-3, symbol Regulator_Linear:HT75xx-1-SOT89
- added C1: 220uF, Capacitor_SMD:CP_Elec_6.3x7.7, symbol Device:C
- added C2, C6: 10uF, Capacitor_SMD:C_0603_1608Metric, symbol Device:C
- added C3, C4, C7 (x2): 100nF, Capacitor_SMD:C_0603_1608Metric, symbol Device:C
- added C5: 22uF, Capacitor_SMD:CP_Elec_6.3x5.4, symbol Device:C
- added D4: 1N5819WS, Diode_SMD:D_SOD-323, symbol Diode:1N5819WS
- added D6 (x2): LED_Small, LED_SMD:LED_0603_1608Metric, symbol Device:LED_Small
- added D7: PMEG6020ER, Diode_SMD:Nexperia_CFP3_SOD-123W, symbol Diode:PMEG6020ER
- added H1, H2: MountingHole, MountingHole:MountingHole_2.5mm, symbol Mechanical:MountingHole
- added J5: Conn_01x06_Socket, Connector_PinSocket_2.54mm:PinSocket_1x06_P2.54mm_Vertical, symbol Connector:Conn_01x06_Socket
- added L1: 10uH, Inductor_SMD:L_Chilisin_BMRA00040415, symbol Device:L
- added Q1, Q3: CSD19537Q3, Package_SON:VSON-8_3.3x3.3mm_P0.65mm_NexFET, symbol Transistor_FET:CSD19537Q3
- added Q2: MMBT3904, Package_TO_SOT_SMD:SOT-23, symbol Transistor_BJT:MMBT3904
- added R3 (x4): 13k, Resistor_SMD:R_0603_1608Metric, symbol Device:R
- added R3: 1k, Resistor_SMD:R_0603_1608Metric, symbol Device:R
- added R4: 4.3k, Resistor_SMD:R_0603_1608Metric, symbol Device:R
- added R7 (x3): 2.2k, Resistor_SMD:R_0603_1608Metric, symbol Device:R
- added TP1, TP2: TestPoint, TestPoint:TestPoint_Pad_D2.0mm, symbol Connector:TestPoint
- added TP3: TestPoint, TestPoint:TestPoint_Loop_D3.50mm_Drill1.4mm_Beaded, symbol Connector:TestPoint
- added U2: ESP32-C3-MINI-1, Espressif:ESP32-C3-MINI-1, symbol Espressif:ESP32-C3-MINI-1
- added U3: AOZ1280CI, Package_TO_SOT_SMD:SOT-23-6, symbol Regulator_Switching:AOZ1280CI
- J1, J2, J3: footprint XT60PW-M:AMASS_XT60PW-M -> Acea:AMASS_XT60PW-F_1x02_P7.20mm_Horizontal
- J4: footprint XT60PW-M:AMASS_XT60PW-M -> Acea:AMASS_XT60PW-M_1x02_P7.20mm_Horizontal
Connections:
- net +12V: now also C1.1, C2.1, C3.1, D4.1 (K), R3.1, R3.1, U3.4 (EN), U3.5 (VIN)
- net +3.3V: now also C5.1, C6.1, C7.1, C7.1, J5.6 (Pin_6), L1.2, R3.1, R3.1, R7.2, U2.3 (3V3)
- net GND: now also C1.2, C2.2, C3.2, C5.2, C6.2, C7.2, C7.2, D6.1 (K), D6.1 (K), D7.2 (A), J5.1 (Pin_1), Q1.1 (S), Q1.2 (S), Q1.3 (S), Q2.2 (E), Q3.1 (S), Q3.2 (S), Q3.3 (S), R4.2, R7.1, TP2.1, U2.1 (GND), U2.11 (GND), U2.14 (GND), U2.2 (GND), U2.36 (GND), U2.37 (GND), U2.38 (GND), U2.39 (GND), U2.40 (GND), U2.41 (GND), U2.42 (GND), U2.43 (GND), U2.44 (GND), U2.45 (GND), U2.46 (GND), U2.47 (GND), U2.48 (GND), U2.49 (GND), U2.50 (GND), U2.51 (GND), U2.52 (GND), U2.53 (GND), U3.2 (GND)
- net at J1.2 (Pin_2), J2.2 (Pin_2), J3.2 (Pin_2): now also D4.2 (A), Q1.5 (D), Q3.5 (D)
- new net: D6.2 (A), R7.1 (x2)
- new net: Q1.4 (G), Q2.3 (C), Q3.4 (G), R3.2
- new net: Q2.1 (B), R3.2
- new net: C4.2, D7.1 (K), L1.1, U3.6 (LX)
- new net: R3.2, R4.1, U3.3 (FB)
- new net: C4.1, U3.1 (BST)
- new net: TP1.1, U2.23 (GPIO9)
- new net: J5.3 (Pin_3), U2.30 (GPIO20/U0RXD)
- new net: J5.4 (Pin_4), U2.31 (GPIO21/U0TXD)
- new net: R3.2, U2.8 (EN/CHIP_PU)
- new net MOSFET: R3.1, U2.6 (GPIO3/ADC1_CH3)
- new net SWITCH: TP3.1, U2.19 (GPIO5/ADC2_CH0)
- new net SYS_LED: R7.2, U2.18 (GPIO4/ADC1_CH4)
- new net VIn: R3.2, R7.2, U2.13 (GPIO1/ADC1_CH1/XTAL_32K_N)
- no-connect marks 0 -> 8
Other:
- note added: "3.3V Available"
- note added: "DC-DC VIN-5V"
- note added: "SYS OK"
- note added: "TTL-UART"
- note added: "Voltage Sense"
- moved on the sheet: J1, J2, J3, J4

Commit message: v0.1 submitted for PCBA
Parts:
- added FID1, FID2, FID3, FID4: Fiducial, Fiducial:Fiducial_0.5mm_Mask1.5mm, symbol Mechanical:Fiducial
- C1: lcsc C99836 -> C340768
- J1, J2, J3: lcsc (none) -> C428722
- J4: lcsc (none) -> C98732
- U2: lcsc (none) -> C5290152
Changed lines of the file:
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@@
+    )
+  )
+  (symbol (lib_id "Mechanical:Fiducial") (at 267.208 39.624 0) (unit 1)
+    (in_bom yes) (on_board yes) (dnp no) (fields_autoplaced)
+    (property "Reference" "FID2" (at 270.51 38.354 0)
+      (effects (font (size 1.27 1.27)) (justify left))
+    )
+    (property "Value" "Fiducial" (at 270.51 40.894 0)
+      (effects (font (size 1.27 1.27)) (justify left))
+    )
+    (property "Footprint" "Fiducial:Fiducial_0.5mm_Mask1.5mm" (at 267.208 39.624 0)
+      (effects (font (size 1.27 1.27)) hide)
+    )
+    (property "Datasheet" "~" (at 267.208 39.624 0)
+      (effects (font (size 1.27 1.27)) hide)
+    )
+    (property "lcsc" "" (at 267.208 39.624 0)
+      (effects (font (size 1.27 1.27)) hide)
+    )
+    (instances
+      (project "JonoBro"
+        (path "/c9de2c96-175d-487c-863d-0ad50f79f798"
+          (reference "FID2") (unit 1)
+        )
+      )
     )
   )
@@
     )
   )
+  (symbol (lib_id "Mechanical:Fiducial") (at 267.208 44.45 0) (unit 1)
+    (in_bom yes) (on_board yes) (dnp no) (fields_autoplaced)
+    (property "Reference" "FID3" (at 270.51 43.18 0)
+      (effects (font (size 1.27 1.27)) (justify left))
+    )
+    (property "Value" "Fiducial" (at 270.51 45.72 0)
+      (effects (font (size 1.27 1.27)) (justify left))
+    )
+    (property "Footprint" "Fiducial:Fiducial_0.5mm_Mask1.5mm" (at 267.208 44.45 0)
+      (effects (font (size 1.27 1.27)) hide)
+    )
+    (property "Datasheet" "~" (at 267.208 44.45 0)
+      (effects (font (size 1.27 1.27)) hide)
+    )
+    (property "lcsc" "" (at 267.208 44.45 0)
+      (effects (font (size 1.27 1.27)) hide)
+    )
+    (instances
+      (project "JonoBro"
+        (path "/c9de2c96-175d-487c-863d-0ad50f79f798"
+          (reference "FID3") (unit 1)
+        )
+      )
+    )
+  )
   (symbol (lib_id "power:GND") (at 86.106 84.074 0) (unit 1)
     (in_bom yes) (on_board yes) (dnp no) (fields_autoplaced)
@@
       (effects (font (size 1.27 1.27)) hide)
     )
-    (property "lcsc" "" (at 241.3 103.378 0)
+    (property "lcsc" "C428722" (at 241.3 103.378 0)
       (effects (font (size 1.27 1.27)) hide)
     )
@@
       (effects (font (size 1.27 1.27)) hide)
     )
-    (property "lcsc" "" (at 241.3 88.138 0)
+    (property "lcsc" "C428722" (at 241.3 88.138 0)
       (effects (font (size 1.27 1.27)) hide)
     )
@@
     )
   )
+  (symbol (lib_id "Mechanical:Fiducial") (at 267.208 49.276 0) (unit 1)
+    (in_bom yes) (on_board yes) (dnp no) (fields_autoplaced)
+    (property "Reference" "FID4" (at 270.51 48.006 0)
+      (effects (font (size 1.27 1.27)) (justify left))
+    )
+    (property "Value" "Fiducial" (at 270.51 50.546 0)
+      (effects (font (size 1.27 1.27)) (justify left))
+    )
+    (property "Footprint" "Fiducial:Fiducial_0.5mm_Mask1.5mm" (at 267.208 49.276 0)
+      (effects (font (size 1.27 1.27)) hide)
+    )
+    (property "Datasheet" "~" (at 267.208 49.276 0)
+      (effects (font (size 1.27 1.27)) hide)
+    )
+    (property "lcsc" "" (at 267.208 49.276 0)
+      (effects (font (size 1.27 1.27)) hide)
+    )
+    (instances
+      (project "JonoBro"
+        (path "/c9de2c96-175d-487c-863d-0ad50f79f798"
+          (reference "FID4") (unit 1)
+        )
+      )
+    )
+  )
   (symbol (lib_id "Device:C") (at 155.702 40.64 0) (unit 1)
     (in_bom yes) (on_board yes) (dnp no) (fields_autoplaced)
@@
       (effects (font (size 1.27 1.27)) hide)
     )
-    (property "lcsc" "" (at 241.3 118.618 0)
+    (property "lcsc" "C428722" (at 241.3 118.618 0)
       (effects (font (size 1.27 1.27)) hide)
     )
@@
   )
   (symbol (lib_id "Espressif:ESP32-C3-MINI-1") (at 102.87 116.586 0) (unit 1)
-    (in_bom yes) (on_board yes) (dnp no) (fields_autoplaced)
+    (in_bom yes) (on_board yes) (dnp no)
     (property "Reference" "U2" (at 77.47 86.106 0)
       (effects (font (size 1.27 1.27)) (justify left))
     )
-    (property "Value" "ESP32-C3-MINI-1" (at 77.47 88.646 0)
+    (property "Value" "ESP32-C3-MINI-1" (at 106.68 88.9 0)
       (effects (font (size 1.27 1.27)) (justify left))
     )
@@
     )
     (property "Datasheet" "https://www.espressif.com/sites/default/files/documentation/esp32-c3-mini-1_datasheet_en.pdf" (at 102.87 154.686 0)
+      (effects (font (size 1.27 1.27)) hide)
+    )
+    (property "lcsc" "C5290152" (at 102.87 116.586 0)
       (effects (font (size 1.27 1.27)) hide)
     )
@@
       (effects (font (size 1.27 1.27)) hide)
     )
-    (property "lcsc" "C99836" (at 29.972 38.1 0)
+    (property "lcsc" "C340768" (at 29.972 38.1 0)
       (effects (font (size 1.27 1.27)) hide)
     )
@@
       (effects (font (size 1.27 1.27)) hide)
     )
-    (property "lcsc" "" (at 25.4 176.022 0)
+    (property "lcsc" "C98732" (at 25.4 176.022 0)
       (effects (font (size 1.27 1.27)) hide)
     )
@@
         )
       )
+    )
+  )
+  (symbol (lib_id "Mechanical:Fiducial") (at 267.208 34.544 0) (unit 1)
+    (in_bom yes) (on_board yes) (dnp no) (fields_autoplaced)
+    (property "Reference" "FID1" (at 270.51 33.274 0)
+      (effects (font (size 1.27 1.27)) (justify left))
+    )
+    (property "Value" "Fiducial" (at 270.51 35.814 0)
+      (effects (font (size 1.27 1.27)) (justify left))
+    )
+    (property "Footprint" "Fiducial:Fiducial_0.5mm_Mask1.5mm" (at 267.208 34.544 0)
+      (effects (font (size 1.27 1.27)) hide)
+    )
+    (property "Datasheet" "~" (at 267.208 34.544 0)
+      (effects (font (size 1.27 1.27)) hide)
+    )
+    (property "lcsc" "" (at 267.208 34.544 0)
+      (effects (font (size 1.27 1.27)) hide)
+    )
+    (instances
+      (project "JonoBro"
+        (path "/c9de2c96-175d-487c-863d-0ad50f79f798"
+          (reference "FID1") (unit 1)
+        )
+      )
