File: hardware/JonoBro.kicad_pcb (KiCad board)
At the start: 2 copper layers, 44.7 x 56.5 mm, 42 parts, among them J1 Conn_01x02_Pin, J2 Conn_01x02_Pin, J3 Conn_01x02_Pin, J4 Conn_01x02_Pin, J5 Conn_01x06_Socket, Q1 CSD19537Q3, Q2 MMBT3904, Q3 CSD19537Q3, U1 AOZ1280CI, U2 ESP32-C3-MINI-1

Commit message: moved things around
Parts:
- added R10: 13k, Resistor_SMD:R_0603_1608Metric, F.Cu at (151.9, 102.2)
- added R11: 13k, Resistor_SMD:R_0603_1608Metric, F.Cu at (140.8, 107.8)
- added R12: 13k, Resistor_SMD:R_0603_1608Metric, F.Cu at (130.6, 117.2)
- FID1, FID2, FID3, FID4: footprint Fiducial:Fiducial_0.5mm_Mask1.5mm -> Fiducial:Fiducial_1mm_Mask2mm
- TP3: footprint TestPoint:TestPoint_Loop_D3.50mm_Drill1.4mm_Beaded -> TestPoint:TestPoint_Loop_D3.80mm_Drill2.5mm
- moved TP2 1.29 mm to (133.8, 118.3)
- moved TP1 0.97 mm to (138.7, 118.2)
- moved R4 0.77 mm to (142.8, 105.1)
- moved R7 0.75 mm to (142.8, 103.5)
- moved C8 0.67 mm to (149.6, 100.8)
- moved R5 0.46 mm to (148.1, 100.9)
- moved D3 0.21 mm to (142.8, 114.3)
- moved R6 0.21 mm to (142.8, 111.0)
Connections:
- U2 pad 22: unconnected-(U2-GPIO8-Pad22) -> Net-(U2-GPIO8)
- U2 pad 5: unconnected-(U2-GPIO2/ADC1_CH2-Pad5) -> Net-(U2-GPIO2/ADC1_CH2)
Routing:
- net Net-(U2-GPIO8): track 0.00 -> 12.8 mm, vias 0 -> 2
- net +3.3V: track 43.1 -> 53.2 mm
- net Net-(U2-GPIO9): track 19.2 -> 26.7 mm
- net Net-(U2-GPIO2/ADC1_CH2): track 0.00 -> 1.65 mm
- net MOSFET: track 21.7 -> 22.3 mm
Other:
- board size 44.7 x 56.5 mm -> 44.7 x 56.9 mm
- board text added: "JonoTron-3000 v0.2"
- board text removed: "JonoTron-3000 v0.1"

Commit message: pcb updates to 0.2
Parts:
- removed FID1, FID2, FID3, FID4: Fiducial, Fiducial:Fiducial_1mm_Mask2mm
- removed J5: Conn_01x06_Socket, Connector_PinSocket_2.54mm:PinSocket_1x06_P2.54mm_Vertical
- added D5: 1N5819WS, Diode_SMD:D_SOD-323, F.Cu at (128.9, 89.3)
- added D6: 1N5819WS, Diode_SMD:D_SOD-323, F.Cu at (154.8, 107.2)
- added D7: 1N5819WS, Diode_SMD:D_SOD-323, F.Cu at (155.0, 86.2)
- added J6: USB_C_Receptacle_USB2.0, Connector_USB:USB_C_Receptacle_HRO_TYPE-C-31-M-12, F.Cu at (121.8, 92.5)
- added Q4: MMBT3904, Package_TO_SOT_SMD:SOT-23, F.Cu at (135.8, 79.0)
- added Q5: CSD19537Q3, Package_SON:VSON-8_3.3x3.3mm_P0.65mm_NexFET, F.Cu at (146.1, 109.6)
- added Q6: CSD19537Q3, Package_SON:VSON-8_3.3x3.3mm_P0.65mm_NexFET, F.Cu at (146.1, 114.5)
- added Q7: MMBT3904, Package_TO_SOT_SMD:SOT-23, F.Cu at (139.6, 79.0)
- added Q8: CSD19537Q3, Package_SON:VSON-8_3.3x3.3mm_P0.65mm_NexFET, F.Cu at (147.9, 88.5)
- added Q9: CSD19537Q3, Package_SON:VSON-8_3.3x3.3mm_P0.65mm_NexFET, F.Cu at (146.5, 93.9)
- added R13: 5.1k, Resistor_SMD:R_0603_1608Metric, F.Cu at (128.8, 91.2)
- added R14: 5.1k, Resistor_SMD:R_0603_1608Metric, F.Cu at (128.8, 94.2)
- added R15: 1k, Resistor_SMD:R_0603_1608Metric, F.Cu at (139.4, 75.8)
- added R16: 13k, Resistor_SMD:R_0603_1608Metric, F.Cu at (136.0, 74.0)
- added R17: 1k, Resistor_SMD:R_0603_1608Metric, F.Cu at (136.0, 75.8)
- added R18: 13k, Resistor_SMD:R_0603_1608Metric, F.Cu at (139.4, 73.8)
- added R19: 13k, Resistor_SMD:R_0603_1608Metric, F.Cu at (123.3, 83.4)
- added TP4: TestPoint, TestPoint:TestPoint_Pad_D1.0mm, F.Cu at (135.8, 71.6)
- added TP5: TestPoint, TestPoint:TestPoint_Pad_D1.0mm, F.Cu at (138.0, 71.6)
- TP1, TP2: footprint TestPoint:TestPoint_Pad_D2.0mm -> TestPoint:TestPoint_Pad_D1.0mm
- moved H2 55.6 mm to (140.0, 125.8)
- moved D2 49.0 mm to (136.2, 65.5), turned to -90 degrees
- moved D3 49.0 mm to (138.2, 65.5), turned to -90 degrees
- moved U2 44.7 mm to (127.0, 73.3), turned to 0 degrees
- moved R3 42.5 mm to (136.2, 68.8), turned to -90 degrees
- moved R6 42.5 mm to (138.2, 68.8), turned to -90 degrees
- moved R10 42.4 mm to (119.3, 75.1), turned to -90 degrees
- moved C8 41.8 mm to (119.3, 72.0)
- moved J1 39.1 mm to (154.2, 100.1), turned to -90 degrees
- moved R5 36.6 mm to (119.3, 78.2), turned to -90 degrees
- moved TP1 35.1 mm to (134.4, 83.4), turned to 90 degrees
- moved TP2 35.0 mm to (136.6, 83.4), turned to -90 degrees
- moved R12 33.7 mm to (132.5, 83.5), turned to 90 degrees
- moved H1 31.7 mm to (151.2, 67.6)
- moved R7 30.2 mm to (120.2, 83.4), turned to 90 degrees
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Connections:
- J1 pad 2: Net-(D4-A) -> Net-(D7-A)
- J2 pad 2: Net-(D4-A) -> Net-(D6-A)
- R8 pad 1: MOSFET -> MOSFET_WS
- U2 pad 16: unconnected-(U2-GPIO10-Pad16) -> MOSFET_WS
- U2 pad 20: unconnected-(U2-GPIO6-Pad20) -> MOSFET_LMR
- U2 pad 21: unconnected-(U2-GPIO7-Pad21) -> MOSFET_RMR
- U2 pad 26: unconnected-(U2-GPIO18/USB_D--Pad26) -> USBD-
- U2 pad 27: unconnected-(U2-GPIO19/USB_D+-Pad27) -> USBD+
- U2 pad 6: MOSFET -> unconnected-(U2-GPIO3/ADC1_CH3-Pad6)
Routing:
- net Net-(Q4-C): track 0.00 -> 116.1 mm, vias 0 -> 3
- net Net-(Q7-C): track 0.00 -> 94.6 mm, vias 0 -> 3
- net SWITCH: track 53.9 -> 8.52 mm, vias 3 -> 0
- net +3.3V: track 53.2 -> 88.1 mm, vias 3 -> 8
- net USBD-: track 0.00 -> 28.5 mm, vias 0 -> 2
- net USBD+: track 0.00 -> 28.1 mm, vias 0 -> 2
- net MOSFET_WS: track 0.00 -> 25.1 mm, vias 0 -> 2
- net MOSFET: track 22.3 -> 0.00 mm, vias 2 -> 0
- net Net-(U2-GPIO9): track 26.7 -> 4.84 mm, vias 2 -> 0
- net SYS_LED: track 5.38 -> 20.7 mm
- net MOSFET_RMR: track 0.00 -> 12.6 mm, vias 0 -> 2
- net MOSFET_LMR: track 0.00 -> 12.5 mm, vias 0 -> 2
- net USB_VBUS: track 0.00 -> 11.2 mm
- net Net-(U2-GPIO8): track 12.8 -> 1.99 mm, vias 2 -> 0
- net Net-(Q1-G): track 14.2 -> 24.0 mm, vias 2 -> 3
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- added copper zone on B.Cu, net Net-(D6-A)
- added copper zone on F.Cu, net Net-(D6-A)
- added copper zone on B.Cu, net Net-(D7-A)
- added copper zone on F.Cu, net Net-(D7-A)
Other:
- board size 44.7 x 56.9 mm -> 44.7 x 65.1 mm
- board text added: "B"
- board text added: "G"
- board text added: "R"
- board text added: "SWITCH"
- board text added: "T"
- board text added: "WINDSCREEN"
- board text removed: "TRIGGER"
- board text removed: "WS"

Commit message: 0.2 wip
Parts:
- removed D3: LED_Small, LED_SMD:LED_0603_1608Metric
- removed R6: 2.2k, Resistor_SMD:R_0603_1608Metric
- added C10: 100nF, Capacitor_SMD:C_0603_1608Metric, F.Cu at (125.5, 83.8)
- added C9: 100nF, Capacitor_SMD:C_0603_1608Metric, F.Cu at (131.7, 83.7)
- TP4, TP5: moved to B.Cu
- moved D6 20.8 mm to (146.5, 126.2), turned to 0 degrees
- moved D7 17.3 mm to (145.1, 100.4), turned to 0 degrees
- moved G*** 13.9 mm to (139.1, 109.3)
- moved Q9 10.8 mm to (146.8, 104.7), turned to 45 degrees
- moved Q3 8.83 mm to (149.7, 84.8), turned to 45 degrees
- moved Q5 8.48 mm to (148.0, 117.9), turned to -45 degrees
- moved Q6 8.33 mm to (147.3, 122.7)
- moved R7 8.32 mm to (128.6, 83.8)
- moved D4 8.26 mm to (147.1, 76.5), turned to -45 degrees
- moved Q8 7.64 mm to (146.8, 96.1)
- moved TP5 7.53 mm to (131.1, 74.7), turned to 180 degrees
- moved D5 7.48 mm to (129.0, 96.8)
- moved H1 6.81 mm to (144.4, 68.0)
- moved R19 6.80 mm to (130.1, 83.7)
- moved Q7 6.63 mm to (139.4, 72.4)
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Connections:
- J1 pad 1: +12V -> Net-(D7-A)
- J1 pad 2: Net-(D7-A) -> +12V
- J2 pad 1: +12V -> Net-(D6-A)
- J2 pad 2: Net-(D6-A) -> +12V
- J3 pad 1: +12V -> Net-(D4-A)
- J3 pad 2: Net-(D4-A) -> +12V
- J4 pad 1: +12V -> GND
- J4 pad 2: GND -> +12V
- U2 pad 18: SYS_LED -> unconnected-(U2-GPIO4/ADC1_CH4-Pad18)
Routing:
- net Net-(Q1-G): track 24.0 -> 68.8 mm
- net Net-(Q4-C): track 116.1 -> 139.6 mm
- net SYS_LED: track 20.7 -> 0.00 mm, vias 2 -> 0
- net Net-(U2-GPIO8): track 1.99 -> 14.0 mm
- net +3.3V: track 88.1 -> 97.6 mm, vias 8 -> 7
- net MOSFET_WS: track 25.1 -> 16.5 mm
- net Net-(Q7-C): track 94.6 -> 100.4 mm
- net SWITCH: track 8.52 -> 14.1 mm
- net Net-(U2-GPIO20/U0RXD): track 7.80 -> 2.34 mm, vias 0 -> 1
- net Net-(U2-GPIO9): track 4.84 -> 9.60 mm
- net USBD-: track 28.5 -> 24.5 mm
- net MOSFET_RMR: track 12.6 -> 16.5 mm
- net VIn: track 4.29 -> 7.15 mm
- net MOSFET_LMR: track 12.5 -> 10.6 mm
- net Net-(Q2-B): track 4.33 -> 6.18 mm
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- removed copper zone on B.Cu, net Net-(D4-A)
Other:
- board text added: "Rx"
- board text added: "Tx"
- board text removed: "PWR"
- board text removed: "R"
- board text removed: "T"

Commit message: 0.2 wip
Parts:
- added H3: MountingHole, MountingHole:MountingHole_4.3mm_M4_Pad_Via, F.Cu at (140.8, 58.8)
- added H4: MountingHole, MountingHole:MountingHole_4.3mm_M4_Pad_Via, F.Cu at (140.8, 133.8)
- added Q10: CSD19537Q3, Package_SON:VSON-8_3.3x3.3mm_P0.65mm_NexFET, F.Cu at (143.3, 78.3)
- added TP6: TestPoint, TestPoint:TestPoint_Pad_D1.0mm, B.Cu at (128.0, 73.0)
- moved D4 3.13 mm to (150.1, 75.6), turned to -90 degrees
- moved Q1 0.69 mm to (146.6, 81.5)
Routing:
- net Net-(Q1-G): track 68.8 -> 73.9 mm, vias 3 -> 4
- net GND: track 3.60 -> 5.03 mm, vias 0 -> 13
- net +12V: track 10.6 -> 9.68 mm, vias 142 -> 149
- net Net-(D4-A): vias 57 -> 65
- added copper zone on B.Cu, net GND
- added copper zone on B.Cu, net Net-(D4-A)
Other:
- board size 44.7 x 65.1 mm -> 44.7 x 85.1 mm

Commit message: 0.2 wip
Parts:
- added SW1: SW_Push, Acea:ALPSALPINE-SKSCLBE010_C115361, B.Cu at (120.0, 103.7)
- added SW2: SW_Push, Acea:ALPSALPINE-SKSCLBE010_C115361, B.Cu at (120.1, 109.5)
- moved Q10 2.23 mm to (144.9, 79.9)
- moved D2 2.02 mm to (136.7, 63.5), turned to 90 degrees
- moved Q1 1.90 mm to (147.9, 82.9)
- moved Q3 1.70 mm to (150.9, 86.0)
- moved D4 1.58 mm to (148.5, 75.8)
- moved Q8 1.28 mm to (146.1, 97.1)
- moved H2 1.22 mm to (139.6, 125.5)
- moved R3 0.95 mm to (134.9, 66.4), turned to -90 degrees
- moved D7 0.60 mm to (145.1, 101.0)
- moved R15 0.40 mm to (139.2, 75.1), turned to 0 degrees
- moved D1 0.40 mm to (128.8, 115.8)
- moved R16 0.20 mm to (136.0, 73.8)
- moved R9 0.10 mm to (134.8, 70.3)
Routing:
- net Net-(U2-GPIO9): track 9.60 -> 52.1 mm, vias 0 -> 1
- net Net-(U2-EN/CHIP_PU): track 2.95 -> 30.0 mm, vias 0 -> 1
- net +3.3V: track 97.6 -> 87.4 mm
- net Net-(Q7-C): track 100.4 -> 93.1 mm
- net GND: track 5.03 -> 8.90 mm, vias 13 -> 22
- net Net-(D2-A): track 1.63 -> 4.03 mm, vias 0 -> 2
- net USBD+: track 27.3 -> 25.0 mm
- net Net-(Q7-B): track 6.09 -> 7.65 mm
- net USBD-: track 24.5 -> 23.0 mm
- net MOSFET_RMR: track 16.5 -> 15.3 mm
- net Net-(Q1-G): track 73.9 -> 72.8 mm
- net Net-(Q4-B): track 3.96 -> 4.91 mm
- net Net-(Q4-C): track 139.6 -> 140.4 mm
- net MOSFET_LMR: track 10.6 -> 9.94 mm
- net +12V: track 9.68 -> 9.43 mm, vias 149 -> 170
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Other:
- board text added: "20V MAX"
- board text added: "BOOT"
- board text added: "RST"
- board text removed: "30V MAX"
