File: hardware/JonoBro.kicad_sch (KiCad schematic)
At the start: 41 parts, among them J1 Conn_01x02_Pin, J2 Conn_01x02_Pin, J3 Conn_01x02_Pin, J4 Conn_01x02_Pin, J5 Conn_01x06_Socket, Q1 CSD19537Q3, Q2 MMBT3904, Q3 CSD19537Q3, U2 ESP32-C3-MINI-1, U3 AOZ1280CI

Commit message: moved things around
Parts:
- added R3 (x3): 13k, Resistor_SMD:R_0603_1608Metric, symbol Device:R
- FID1, FID2, FID3, FID4: footprint Fiducial:Fiducial_0.5mm_Mask1.5mm -> Fiducial:Fiducial_1mm_Mask2mm
- TP3: footprint TestPoint:TestPoint_Loop_D3.50mm_Drill1.4mm_Beaded -> TestPoint:TestPoint_Loop_D3.80mm_Drill2.5mm
Connections:
- net +3.3V: now also R3.1, R3.1, R3.1
- net at U2.22 (GPIO8): now also R3.2
- net at TP1.1, U2.23 (GPIO9): now also R3.2
- net at U2.5 (GPIO2/ADC1_CH2): now also R3.2
Other:
- note added: "GPIO8 requires pullup GPIO2 requires pullup GPIO9 requires pullup(short to GND for UART/USB bootloader)"
- title: (none) -> JonoTron-3000
- moved on the sheet: TP1, TP2

Commit message: pcb updates to 0.2
Parts:
- removed FID1, FID2, FID3, FID4: Fiducial, Fiducial:Fiducial_1mm_Mask2mm, symbol Mechanical:Fiducial
- removed J5: Conn_01x06_Socket, Connector_PinSocket_2.54mm:PinSocket_1x06_P2.54mm_Vertical, symbol Connector:Conn_01x06_Socket
- added D4 (x3): 1N5819WS, Diode_SMD:D_SOD-323, symbol Diode:1N5819WS
- added J3: USB_C_Receptacle_USB2.0, Connector_USB:USB_C_Receptacle_HRO_TYPE-C-31-M-12, symbol hardware_nrf52840_pa_beacon_hat:USB_C_Receptacle_USB2.0-Connector
- added Q4, Q7: MMBT3904, Package_TO_SOT_SMD:SOT-23, symbol Transistor_BJT:MMBT3904
- added Q5, Q6, Q8, Q9: CSD19537Q3, Package_SON:VSON-8_3.3x3.3mm_P0.65mm_NexFET, symbol Transistor_FET:CSD19537Q3
- added R3 (x3): 13k, Resistor_SMD:R_0603_1608Metric, symbol Device:R
- added R3 (x2): 1k, Resistor_SMD:R_0603_1608Metric, symbol Device:R
- added R7, R8: 5.1k, Resistor_SMD:R_0603_1608Metric, symbol Device:R
- added TP4, TP5: TestPoint, TestPoint:TestPoint_Pad_D1.0mm, symbol Connector:TestPoint
- TP1, TP2: footprint TestPoint:TestPoint_Pad_D2.0mm -> TestPoint:TestPoint_Pad_D1.0mm
Connections:
- net +12V: now also D4.1 (K), D4.1 (K), D4.1 (K), R3.1, R3.1, R3.1
- net GND: now also J3.A1 (GND), J3.A12 (GND), J3.B1 (GND), J3.B12 (GND), J3.S1 (SHIELD), Q4.2 (E), Q5.1 (S), Q5.2 (S), Q5.3 (S), Q6.1 (S), Q6.2 (S), Q6.3 (S), Q7.2 (E), Q8.1 (S), Q8.2 (S), Q8.3 (S), Q9.1 (S), Q9.2 (S), Q9.3 (S), R7.1, R8.1
- net SWITCH: now also R3.2
- net at D4.2 (A), J3.2 (Pin_2), Q1.5 (D)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: no longer J1.2 (Pin_2), J2.2 (Pin_2)
- net MOSFET_WS: now reaches U2.16 (GPIO10)
- net MOSFET_WS: now also R3.1
- net MOSFET_LMR: now reaches U2.20 (GPIO6)
- net MOSFET_LMR: now also R3.1
- net MOSFET_RMR: now reaches U2.21 (GPIO7)
- net MOSFET_RMR: now also R3.1
- net USBD-: now reaches U2.26 (GPIO18/USB_D-)
- net USBD-: now also J3.A7 (D-), J3.B7 (D-)
- net USBD+: now reaches U2.27 (GPIO19/USB_D+)
- net USBD+: now also J3.A6 (D+), J3.B6 (D+)
- net at U2.30 (GPIO20/U0RXD): now also TP5.1
- net at U2.31 (GPIO21/U0TXD): now also TP4.1
- net MOSFET: no longer names the net of U2.6 (GPIO3/ADC1_CH3)
- net MOSFET: no longer R3.1
- new net: J3.A5 (CC1), R7.2
- new net: J3.B5 (CC2), R8.2
- new net: Q7.3 (C), Q8.4 (G), Q9.4 (G), R3.2
- new net: D4.2 (A), J1.2 (Pin_2), Q8.5 (D), Q9.5 (D)
- new net: D4.2 (A), J2.2 (Pin_2), Q5.5 (D), Q6.5 (D)
- new net: Q4.1 (B), R3.2
- new net: Q7.1 (B), R3.2
- new net: Q4.3 (C), Q5.4 (G), Q6.4 (G), R3.2
- new net USB_VBUS: D4.2 (A), J3.A4 (VBUS), J3.A9 (VBUS), J3.B4 (VBUS), J3.B9 (VBUS)
- no-connect marks 8 -> 4
Other:
- note added: "USB-C"
- note removed: "TTL-UART"
- moved on the sheet: C1, C2, C3, C4, C5, C6, C7, D4, D6, D7, H1, H2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

Commit message: WIP, mostly working v0.1
Other:
- note added: "Bootstrapping:"

Commit message: 0.2 wip
Parts:
- removed D6: LED_Small, LED_SMD:LED_0603_1608Metric, symbol Device:LED_Small
- removed R7: 2.2k, Resistor_SMD:R_0603_1608Metric, symbol Device:R
- added C7 (x2): 100nF, Capacitor_SMD:C_0603_1608Metric, symbol Device:C
Connections:
- net +12V: now also J1.2 (Pin_2), J2.2 (Pin_2), J3.2 (Pin_2), J4.2 (Pin_2), C7.1; no longer J1.1 (Pin_1), J2.1 (Pin_1), J3.1 (Pin_1), J4.1 (Pin_1)
- net GND: now also J4.1 (Pin_1), C7.2; no longer J4.2 (Pin_2)
- net SWITCH: now also C7.2
- net VIn: now also C7.1
- net at D4.2 (A), Q8.5 (D), Q9.5 (D): now also J1.1 (Pin_1); no longer J1.2 (Pin_2)
- net at D4.2 (A), Q5.5 (D), Q6.5 (D): now also J2.1 (Pin_1); no longer J2.2 (Pin_2)
- net at D4.2 (A), Q1.5 (D), Q3.5 (D): now also J3.1 (Pin_1); no longer J3.2 (Pin_2)
- net SYS_LED: no longer names the net of U2.18 (GPIO4/ADC1_CH4)
- no-connect marks 4 -> 5
Other:
- note removed: "SYS OK"

Commit message: 0.2 wip
Parts:
- added H3, H4: MountingHole, MountingHole:MountingHole_4.3mm_M4_Pad_Via, symbol Mechanical:MountingHole
- added Q10: CSD19537Q3, Package_SON:VSON-8_3.3x3.3mm_P0.65mm_NexFET, symbol Transistor_FET:CSD19537Q3
- added TP6: TestPoint, TestPoint:TestPoint_Pad_D1.0mm, symbol Connector:TestPoint
Connections:
- net GND: now also Q10.1 (S), Q10.2 (S), Q10.3 (S), TP6.1
- net at Q1.4 (G), Q2.3 (C), Q3.4 (G)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: now also Q10.4 (G)
- net at D4.2 (A), J3.1 (Pin_1), Q1.5 (D)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: now also Q10.5 (D)
Changed lines of the file:
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@@
   (junction (at 75.692 95.25) (diameter 0) (color 0 0 0 0)
   )
+  (junction (at 359.918 63.881) (diameter 0) (color 0 0 0 0)
+  )
   (junction (at 363.601 110.49) (diameter 0) (color 0 0 0 0)
   )
@@
   (junction (at 67.056 246.38) (diameter 0) (color 0 0 0 0)
   )
+  (junction (at 371.856 44.196) (diameter 0) (color 0 0 0 0)
+  )
   (junction (at 360.045 100.076) (diameter 0) (color 0 0 0 0)
   )
@@
     (stroke (width 0) (type default))
   )
+  (wire (pts (xy 386.842 74.295) (xy 386.842 44.196))
+    (stroke (width 0) (type default))
+  )
   (wire (pts (xy 339.979 133.858) (xy 339.979 135.382))
     (stroke (width 0) (type default))
@@
     (stroke (width 0) (type default))
   )
+  (wire (pts (xy 386.842 86.995) (xy 386.842 84.455))
+    (stroke (width 0) (type default))
+  )
   (wire (pts (xy 372.237 185.928) (xy 372.237 208.28))
     (stroke (width 0) (type default))
@@
     (stroke (width 0) (type default))
   )
+  (wire (pts (xy 183.134 156.972) (xy 183.134 155.702))
+    (stroke (width 0) (type default))
+  )
   (wire (pts (xy 363.601 183.134) (xy 363.601 185.928))
     (stroke (width 0) (type default))
@@
     (stroke (width 0) (type default))
   )
+  (wire (pts (xy 359.918 63.881) (xy 364.236 63.881))
+    (stroke (width 0) (type default))
+  )
   (wire (pts (xy 359.664 26.035) (xy 363.22 26.035))
     (stroke (width 0) (type default))
@@
     (stroke (width 0) (type default))
   )
-  (wire (pts (xy 355.6 63.881) (xy 364.236 63.881))
+  (wire (pts (xy 355.6 63.881) (xy 359.918 63.881))
     (stroke (width 0) (type default))
   )
@@
     (stroke (width 0) (type default))
   )
+  (wire (pts (xy 371.856 44.196) (xy 371.856 58.801))
+    (stroke (width 0) (type default))
+  )
   (wire (pts (xy 339.598 59.817) (xy 355.6 59.817))
     (stroke (width 0) (type default))
@@
     (stroke (width 0) (type default))
   )
+  (wire (pts (xy 359.918 79.375) (xy 359.918 63.881))
+    (stroke (width 0) (type default))
+  )
   (wire (pts (xy 363.601 110.49) (xy 363.601 118.872))
     (stroke (width 0) (type default))
@@
     (stroke (width 0) (type default))
   )
+  (wire (pts (xy 379.222 79.375) (xy 359.918 79.375))
+    (stroke (width 0) (type default))
+  )
   (wire (pts (xy 339.979 131.826) (xy 339.979 133.858))
     (stroke (width 0) (type default))
@@
     (stroke (width 0) (type default))
   )
+  (wire (pts (xy 386.842 44.196) (xy 371.856 44.196))
+    (stroke (width 0) (type default))
+  )
   (wire (pts (xy 363.601 110.49) (xy 372.237 110.49))
     (stroke (width 0) (type default))
@@
     (stroke (width 0) (type default))
   )
-  (wire (pts (xy 371.856 36.449) (xy 371.856 58.801))
+  (wire (pts (xy 371.856 36.449) (xy 371.856 44.196))
     (stroke (width 0) (type default))
   )
@@
     )
   )
+  (symbol (lib_id "Transistor_FET:CSD19537Q3") (at 384.302 79.375 0) (unit 1)
+    (in_bom yes) (on_board yes) (dnp no)
+    (property "Reference" "Q10" (at 382.778 73.025 0)
+      (effects (font (size 1.27 1.27)) (justify left))
+    )
+    (property "Value" "CSD19537Q3" (at 389.382 83.439 0)
+      (effects (font (size 1.27 1.27)) (justify left))
+    )
+    (property "Footprint" "Package_SON:VSON-8_3.3x3.3mm_P0.65mm_NexFET" (at 389.382 81.28 0)
+      (effects (font (size 1.27 1.27) italic) (justify left) hide)
+    )
+    (property "Datasheet" "http://www.ti.com/lit/ds/symlink/csd19537q3.pdf" (at 384.302 79.375 90)
+      (effects (font (size 1.27 1.27)) (justify left) hide)
+    )
+    (property "lcsc" "C315567" (at 384.302 79.375 0)
+      (effects (font (size 1.27 1.27)) hide)
+    )
+    (pin "1")
+    (pin "2")
+    (pin "3")
+    (pin "4")
+    (pin "5")
+    (instances
+      (project "JonoBro"
+        (path "/c9de2c96-175d-487c-863d-0ad50f79f798"
+          (reference "Q10") (unit 1)
+        )
+      )
+    )
+  )
   (symbol (lib_id "power:GND") (at 44.196 265.43 0) (unit 1)
     (in_bom yes) (on_board yes) (dnp no)
@@
     )
   )
+  (symbol (lib_id "Mechanical:MountingHole") (at 246.761 269.621 0) (unit 1)
+    (in_bom yes) (on_board yes) (dnp no) (fields_autoplaced)
+    (property "Reference" "H4" (at 249.809 268.351 0)
+      (effects (font (size 1.27 1.27)) (justify left))
+    )
+    (property "Value" "MountingHole" (at 249.809 270.891 0)
+      (effects (font (size 1.27 1.27)) (justify left))
+    )
+    (property "Footprint" "MountingHole:MountingHole_4.3mm_M4_Pad_Via" (at 246.761 269.621 0)
+      (effects (font (size 1.27 1.27)) hide)
+    )
+    (property "Datasheet" "~" (at 246.761 269.621 0)
+      (effects (font (size 1.27 1.27)) hide)
+    )
+    (property "lcsc" "" (at 246.761 269.621 0)
+      (effects (font (size 1.27 1.27)) hide)
+    )
+    (instances
+      (project "JonoBro"
+        (path "/c9de2c96-175d-487c-863d-0ad50f79f798"
+          (reference "H4") (unit 1)
+        )
+      )
+    )
+  )
   (symbol (lib_id "power:GND") (at 149.606 62.992 0) (unit 1)
     (in_bom yes) (on_board yes) (dnp no)
@@
       (effects (font (size 1.27 1.27)) (justify left))
     )
-    (property "Value" "CSD19537Q3" (at 374.396 67.945 0)
+    (property "Value" "CSD19537Q3" (at 373.634 67.945 0)
       (effects (font (size 1.27 1.27)) (justify left))
     )
@@
     )
   )
+  (symbol (lib_id "Connector:TestPoint") (at 183.134 155.702 0) (unit 1)
+    (in_bom yes) (on_board yes) (dnp no) (fields_autoplaced)
+    (property "Reference" "TP6" (at 185.674 151.13 0)
+      (effects (font (size 1.27 1.27)) (justify left))
+    )
+    (property "Value" "TestPoint" (at 185.674 153.67 0)
+      (effects (font (size 1.27 1.27)) (justify left))
+    )
+    (property "Footprint" "TestPoint:TestPoint_Pad_D1.0mm" (at 188.214 155.702 0)
+      (effects (font (size 1.27 1.27)) hide)
+    )
+    (property "Datasheet" "~" (at 188.214 155.702 0)
+      (effects (font (size 1.27 1.27)) hide)
+    )
+    (property "lcsc" "" (at 183.134 155.702 0)
+      (effects (font (size 1.27 1.27)) hide)
+    )
+    (pin "1")
+    (instances
+      (project "JonoBro"
+        (path "/c9de2c96-175d-487c-863d-0ad50f79f798"
+          (reference "TP6") (unit 1)
+        )
+      )
+    )
+  )
   (symbol (lib_id "Diode:1N5819WS") (at 62.611 40.386 90) (unit 1)
     (in_bom yes) (on_board yes) (dnp no) (fields_autoplaced)
@@
     )
   )
+  (symbol (lib_id "Mechanical:MountingHole") (at 246.761 263.525 0) (unit 1)
+    (in_bom yes) (on_board yes) (dnp no) (fields_autoplaced)
+    (property "Reference" "H3" (at 249.809 262.255 0)
+      (effects (font (size 1.27 1.27)) (justify left))
+    )
+    (property "Value" "MountingHole" (at 249.809 264.795 0)
+      (effects (font (size 1.27 1.27)) (justify left))
+    )
+    (property "Footprint" "MountingHole:MountingHole_4.3mm_M4_Pad_Via" (at 246.761 263.525 0)
+      (effects (font (size 1.27 1.27)) hide)
+    )
+    (property "Datasheet" "~" (at 246.761 263.525 0)
+      (effects (font (size 1.27 1.27)) hide)
+    )
+    (property "lcsc" "" (at 246.761 263.525 0)
+      (effects (font (size 1.27 1.27)) hide)
+    )
+    (instances
+      (project "JonoBro"
+        (path "/c9de2c96-175d-487c-863d-0ad50f79f798"
+          (reference "H3") (unit 1)
+        )
+      )
+    )
+  )
   (symbol (lib_id "power:+3.3V") (at 75.692 95.25 0) (unit 1)
     (in_bom yes) (on_board yes) (dnp no)
@@
     )
   )
+  (symbol (lib_id "power:GND") (at 183.134 156.972 0) (unit 1)
+    (in_bom yes) (on_board yes) (dnp no) (fields_autoplaced)
+    (property "Reference" "#PWR046" (at 183.134 163.322 0)
+      (effects (font (size 1.27 1.27)) hide)
+    )
+    (property "Value" "GND" (at 183.134 161.29 0)
+      (effects (font (size 1.27 1.27)))
+    )
+    (property "Footprint" "" (at 183.134 156.972 0)
+      (effects (font (size 1.27 1.27)) hide)
+    )
+    (property "Datasheet" "" (at 183.134 156.972 0)
+      (effects (font (size 1.27 1.27)) hide)
+    )
+    (pin "1")
+    (instances
+      (project "JonoBro"
+        (path "/c9de2c96-175d-487c-863d-0ad50f79f798"
+          (reference "#PWR046") (unit 1)
+        )
+      )
+    )
+  )
   (symbol (lib_id "power:GND") (at 371.856 71.501 0) (unit 1)
     (in_bom yes) (on_board yes) (dnp no) (fields_autoplaced)
@@
         )
       )
+    )
+  )
+  (symbol (lib_id "power:GND") (at 386.842 86.995 0) (unit 1)
+    (in_bom yes) (on_board yes) (dnp no) (fields_autoplaced)
+    (property "Reference" "#PWR025" (at 386.842 93.345 0)
+      (effects (font (size 1.27 1.27)) hide)
+    )
+    (property "Value" "GND" (at 386.842 92.075 0)
+      (effects (font (size 1.27 1.27)))
+    )
+    (property "Footprint" "" (at 386.842 86.995 0)
+      (effects (font (size 1.27 1.27)) hide)
+    )
+    (property "Datasheet" "" (at 386.842 86.995 0)
+      (effects (font (size 1.27 1.27)) hide)
+    )
+    (pin "1")
+    (instances
+      (project "JonoBro"
+        (path "/c9de2c96-175d-487c-863d-0ad50f79f798"
+          (reference "#PWR025") (unit 1)
+        )
+      )

Commit message: 0.2 wip
Parts:
- added SW1, SW2: SW_Push, Acea:ALPSALPINE-SKSCLBE010_C115361, symbol Switch:SW_Push
Connections:
- net GND: now also SW1.2, SW2.2
- net at R3.2, TP1.1, U2.23 (GPIO9): now also SW2.1
- net at R3.2, U2.8 (EN/CHIP_PU): now also SW1.1
Changed lines of the file:
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@@
   (junction (at 359.918 63.881) (diameter 0) (color 0 0 0 0)
   )
+  (junction (at 142.24 155.702) (diameter 0) (color 0 0 0 0)
+  )
   (junction (at 363.601 110.49) (diameter 0) (color 0 0 0 0)
   )
@@
   (junction (at 119.761 47.752) (diameter 0) (color 0 0 0 0)
   )
+  (junction (at 62.23 112.522) (diameter 0) (color 0 0 0 0)
+  )
   (junction (at 339.598 59.817) (diameter 0) (color 0 0 0 0)
   )
@@
     (stroke (width 0) (type default))
   )
+  (wire (pts (xy 142.24 166.37) (xy 142.24 155.702))
+    (stroke (width 0) (type default))
+  )
   (wire (pts (xy 363.601 185.928) (xy 372.237 185.928))
     (stroke (width 0) (type default))
@@
     (stroke (width 0) (type default))
   )
+  (wire (pts (xy 147.32 155.702) (xy 155.448 155.702))
+    (stroke (width 0) (type default))
+  )
   (wire (pts (xy 372.237 185.928) (xy 372.237 208.28))
     (stroke (width 0) (type default))
@@
     (stroke (width 0) (type default))
   )
+  (wire (pts (xy 58.547 112.522) (xy 62.23 112.522))
+    (stroke (width 0) (type default))
+  )
   (wire (pts (xy 68.326 246.38) (xy 67.056 246.38))
     (stroke (width 0) (type default))
@@
     (stroke (width 0) (type default))
   )
+  (wire (pts (xy 120.396 155.702) (xy 142.24 155.702))
+    (stroke (width 0) (type default))
+  )
   (wire (pts (xy 47.371 45.212) (xy 62.611 45.212))
     (stroke (width 0) (type default))
@@
     (stroke (width 0) (type default))
   )
+  (wire (pts (xy 142.24 155.702) (xy 147.32 155.702))
+    (stroke (width 0) (type default))
+  )
   (wire (pts (xy 156.718 138.176) (xy 159.639 138.176))
     (stroke (width 0) (type default))
@@
     (stroke (width 0) (type default))
   )
-  (wire (pts (xy 147.32 155.702) (xy 155.448 155.702))
-    (stroke (width 0) (type default))
-  )
   (wire (pts (xy 75.946 234.95) (xy 75.946 233.68))
     (stroke (width 0) (type default))
@@
     (stroke (width 0) (type default))
   )
-  (wire (pts (xy 120.396 155.702) (xy 147.32 155.702))
-    (stroke (width 0) (type default))
-  )
   (wire (pts (xy 92.456 95.25) (xy 75.692 95.25))
     (stroke (width 0) (type default))
@@
     )
   )
+  (symbol (lib_id "Switch:SW_Push") (at 53.467 112.522 0) (mirror y) (unit 1)
+    (in_bom yes) (on_board yes) (dnp no) (fields_autoplaced)
+    (property "Reference" "SW1" (at 53.467 104.14 0)
+      (effects (font (size 1.27 1.27)))
+    )
+    (property "Value" "SW_Push" (at 53.467 106.68 0)
+      (effects (font (size 1.27 1.27)))
+    )
+    (property "Footprint" "Acea:ALPSALPINE-SKSCLBE010_C115361" (at 53.467 107.442 0)
+      (effects (font (size 1.27 1.27)) hide)
+    )
+    (property "Datasheet" "~" (at 53.467 107.442 0)
+      (effects (font (size 1.27 1.27)) hide)
+    )
+    (property "lcsc" "C115361" (at 53.467 112.522 0)
+      (effects (font (size 1.27 1.27)) hide)
+    )
+    (pin "1")
+    (pin "2")
+    (instances
+      (project "JonoBro"
+        (path "/c9de2c96-175d-487c-863d-0ad50f79f798"
+          (reference "SW1") (unit 1)
+        )
+      )
+    )
+  )
   (symbol (lib_id "power:GND") (at 44.196 265.43 0) (unit 1)
     (in_bom yes) (on_board yes) (dnp no)
@@
     )
   )
+  (symbol (lib_id "power:GND") (at 48.387 112.522 0) (mirror y) (unit 1)
+    (in_bom yes) (on_board yes) (dnp no) (fields_autoplaced)
+    (property "Reference" "#PWR048" (at 48.387 118.872 0)
+      (effects (font (size 1.27 1.27)) hide)
+    )
+    (property "Value" "GND" (at 48.387 116.84 0)
+      (effects (font (size 1.27 1.27)))
+    )
+    (property "Footprint" "" (at 48.387 112.522 0)
+      (effects (font (size 1.27 1.27)) hide)
+    )
+    (property "Datasheet" "" (at 48.387 112.522 0)
+      (effects (font (size 1.27 1.27)) hide)
+    )
+    (pin "1")
+    (instances
+      (project "JonoBro"
+        (path "/c9de2c96-175d-487c-863d-0ad50f79f798"
+          (reference "#PWR048") (unit 1)
+        )
+      )
+    )
+  )
   (symbol (lib_id "Mechanical:MountingHole") (at 269.113 263.652 0) (unit 1)
     (in_bom yes) (on_board yes) (dnp no) (fields_autoplaced)
@@
     )
   )
+  (symbol (lib_id "power:GND") (at 152.4 166.37 0) (unit 1)
+    (in_bom yes) (on_board yes) (dnp no) (fields_autoplaced)
+    (property "Reference" "#PWR047" (at 152.4 172.72 0)
+      (effects (font (size 1.27 1.27)) hide)
+    )
+    (property "Value" "GND" (at 152.4 170.688 0)
+      (effects (font (size 1.27 1.27)))
+    )
+    (property "Footprint" "" (at 152.4 166.37 0)
+      (effects (font (size 1.27 1.27)) hide)
+    )
+    (property "Datasheet" "" (at 152.4 166.37 0)
+      (effects (font (size 1.27 1.27)) hide)
+    )
+    (pin "1")
+    (instances
+      (project "JonoBro"
+        (path "/c9de2c96-175d-487c-863d-0ad50f79f798"
+          (reference "#PWR047") (unit 1)
+        )
+      )
+    )
+  )
   (symbol (lib_id "Device:R") (at 140.462 134.112 0) (unit 1)
     (in_bom yes) (on_board yes) (dnp no)
@@
         )
       )
+    )
+  )
+  (symbol (lib_id "Switch:SW_Push") (at 147.32 166.37 0) (unit 1)
+    (in_bom yes) (on_board yes) (dnp no) (fields_autoplaced)
+    (property "Reference" "SW2" (at 147.32 158.75 0)
+      (effects (font (size 1.27 1.27)))
+    )
+    (property "Value" "SW_Push" (at 147.32 161.29 0)
+      (effects (font (size 1.27 1.27)))
+    )
+    (property "Footprint" "Acea:ALPSALPINE-SKSCLBE010_C115361" (at 147.32 161.29 0)
+      (effects (font (size 1.27 1.27)) hide)
+    )
+    (property "Datasheet" "~" (at 147.32 161.29 0)
+      (effects (font (size 1.27 1.27)) hide)
+    )
+    (property "lcsc" "C115361" (at 147.32 166.37 0)
+      (effects (font (size 1.27 1.27)) hide)
+    )
+    (pin "1")
+    (pin "2")
+    (instances
+      (project "JonoBro"
+        (path "/c9de2c96-175d-487c-863d-0ad50f79f798"
+          (reference "SW2") (unit 1)
+        )
+      )
