File: hardware/v0_2/JonoBro.kicad_pcb (KiCad board)
At the start: 2 copper layers, 44.7 x 85.1 mm, 65 parts, among them J1 Conn_01x02_Pin, J2 Conn_01x02_Pin, J3 Conn_01x02_Pin, J4 Conn_01x02_Pin, J6 USB_C_Receptacle_USB2.0, Q1 CSD19537Q3, Q10 CSD19537Q3, Q2 MMBT3904, Q3 CSD19537Q3, Q4 MMBT3904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

Commit message: v0.2 complete JLCPCB
Parts:
- removed R3: 2.2k, Resistor_SMD:R_0603_1608Metric
- added C11: 100nF, Capacitor_SMD:C_0603_1608Metric, F.Cu at (136.0, 72.2)
- added TP8: TestPoint, TestPoint:TestPoint_Pad_D1.0mm, F.Cu at (137.5, 83.5)
- D2: value LED_Small -> WS2812-2020; footprint LED_SMD:LED_0603_1608Metric -> LED_SMD:LED_WS2812B-2020_PLCC4_2.0x2.0mm
- moved G*** 20.3 mm to (138.6, 89.0)
- moved D2 6.51 mm to (135.9, 70.0), turned to 180 degrees
- moved R8 3.91 mm to (136.4, 66.3)
- moved R9 3.91 mm to (134.8, 66.3)
- moved D4 0.82 mm to (147.8, 76.1), turned to -45 degrees
- moved H2 0.65 mm to (140.2, 125.5)
- moved TP5 0.46 mm to (131.2, 74.2)
- moved TP4 0.34 mm to (131.1, 72.6)
- moved TP1 0.30 mm to (134.2, 85.5)
- moved TP2 0.30 mm to (134.2, 83.5)
Connections:
- D2 pad 1: GND -> unconnected-(D2-DO-Pad1)
- D2 pad 2: Net-(D2-A) -> GND
- U2 pad 18: unconnected-(U2-GPIO4/ADC1_CH4-Pad18) -> PXL
- U2 pad 6: unconnected-(U2-GPIO3/ADC1_CH3-Pad6) -> PXL_PWR
Routing:
- net PXL_PWR: track 0.00 -> 21.3 mm, vias 0 -> 2
- net +3.3V: track 87.4 -> 66.7 mm, vias 7 -> 6
- net PXL: track 0.00 -> 17.1 mm, vias 0 -> 2
- net +12V: track 9.43 -> 17.0 mm, vias 170 -> 158
- net Net-(Q7-C): track 93.1 -> 99.0 mm
- net MOSFET_WS: track 16.2 -> 20.4 mm
- net Net-(D2-A): track 4.03 -> 0.00 mm, vias 2 -> 0
- net Net-(Q2-B): track 6.18 -> 5.51 mm
- net Net-(D7-A): vias 70 -> 67
- net Net-(D6-A): vias 73 -> 72
- net Net-(D4-A): vias 65 -> 61
- net GND: vias 22 -> 26
Other:
- board text added: "12V"
- board text added: "BOOT/ TRIGGER"
- board text added: "TRIGGER"
- board text removed: "BOOT"
- board text removed: "SWITCH"

Commit message: WIP
Parts:
- moved TP3 0.15 mm to (122.2, 84.4)
Connections:
- C9 pad 1: +12V -> +3.3V
- R19 pad 1: +12V -> +3.3V
Routing:
- net +3.3V: track 66.7 -> 69.9 mm
- net Net-(U2-GPIO8): track 14.0 -> 13.5 mm
- net +12V: track 17.0 -> 16.5 mm, vias 158 -> 157
- net GND: vias 26 -> 27
Other:
- board text added: "JonoTron-3000 v0.3"
- board text removed: "JonoTron-3000 v0.2"

Commit message: board updates
Parts:
- removed R19: 13k, Resistor_SMD:R_0603_1608Metric
- moved C9 1.52 mm to (130.2, 83.8)
Connections:
- C9 pad 1: +3.3V -> SWITCH
- C9 pad 2: SWITCH -> GND
Routing:
- net +3.3V: track 69.9 -> 66.7 mm
- net Net-(U2-GPIO8): track 13.5 -> 11.0 mm
- net SWITCH: track 14.1 -> 12.8 mm
- net Net-(U2-GPIO9): track 52.3 -> 51.3 mm
