File: hardware/v0_2/JonoBro.kicad_sch (KiCad schematic)
At the start: 64 parts, among them J1 Conn_01x02_Pin, J2 Conn_01x02_Pin, J3 Conn_01x02_Pin, J3 USB_C_Receptacle_USB2.0, J4 Conn_01x02_Pin, Q1 CSD19537Q3, Q10 CSD19537Q3, Q2 MMBT3904, Q3 CSD19537Q3, Q4 MMBT3904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

Commit message: v0.2 complete JLCPCB
Parts:
- removed D6: LED_Small, LED_SMD:LED_0603_1608Metric, symbol Device:LED_Small
- removed R7: 2.2k, Resistor_SMD:R_0603_1608Metric, symbol Device:R
- added C11: 100nF, Capacitor_SMD:C_0603_1608Metric, symbol Device:C_Small
- added D2: WS2812-2020, LED_SMD:LED_WS2812B-2020_PLCC4_2.0x2.0mm, symbol ws2812-2020-breakout-rescue:WS2812-2020-LED
- added TP8: TestPoint, TestPoint:TestPoint_Pad_D1.0mm, symbol Connector:TestPoint
Connections:
- net +12V: now also TP8.1
- net GND: now also C11.2, D2.2 (GND)
- net PXL: now reaches U2.18 (GPIO4/ADC1_CH4)
- net PXL: now also D2.3 (DI)
- net PXL_PWR: now reaches U2.6 (GPIO3/ADC1_CH3)
- net PXL_PWR: now also C11.1, D2.4 (VDD)
- no-connect marks 5 -> 4
Other:
- note added: "NeoPixel"
- note added: "NeoPixel LED"
- note removed: "3.3V Available"

Commit message: WIP
Connections:
- net +12V: no longer C7.1, R3.1
- net +3.3V: now also C7.1, R3.1
Other:
- note added: "Switched from 12v to 3.3 in v0.3"
- moved on the sheet: C7, R3, TP3

Commit message: board updates
Parts:
- removed R3: 13k, Resistor_SMD:R_0603_1608Metric, symbol Device:R
Connections:
- net +3.3V: no longer C7.1
- net GND: now also C7.2
- net SWITCH: now also C7.1; no longer C7.2
Other:
- note added: "12v pullup was removed in v0.3"
- note removed: "Switched from 12v to 3.3 in v0.3"
- moved on the sheet: C7, TP3
